File: sweepv2.kicad_pcb (KiCad board)
At the start: 2 copper layers, 216.9 x 86.1 mm, 52 parts, among them J1 AudioJack4dpb, J2 AudioJack4dpb, SW10 SW_Push, SW11 SW_Push, SW11_r1 SW_Push, SW12 SW_Push, SW12_r1 SW_Push, SW13_r1 SW_Push, SW14 SW_Push, SW15 SW_Push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

Commit message: Touch Ups
Parts:
- removed the G*** at (84.1, 85.3)
- added G***: LOGO, LOGO, F.Cu at (83.8, 84.8)
Other:
- board text removed: "Sweep v 2.2"
